Commit message: Added Depth and RGBD Odometry

File: jackal_description/urdf/jackal.urdf.xacro (robot description, xacro)
@@ -232,5 +232,4 @@
 </link>
 <gazebo reference="camera_link">
-<material>Gazebo/Green</material>
   <sensor name="realsense_rgbd" type="depth">
     <always_on>true</always_on>
@@ -250,21 +249,27 @@
       </clip>
     </camera>
-    <!-- RGB Plugin -->
-    <plugin name="camera_controller_color" filename="libgazebo_ros_camera.so">
+    <plugin name="camera_controller" filename="libgazebo_ros_openni_kinect.so">
+      <baseline>0.2</baseline>
       <alwaysOn>true</alwaysOn>
       <updateRate>30.0</updateRate>
-      <cameraName>camera/color</cameraName>
+      <cameraName>camera</cameraName>
       <imageTopicName>color/image_raw</imageTopicName>
       <cameraInfoTopicName>color/camera_info</cameraInfoTopicName>
-      <frameName>camera_link</frameName>
-    </plugin>
-    <!-- Depth Plugin -->
-    <plugin name="camera_controller_depth" filename="libgazebo_ros_depth_camera.so">
-      <alwaysOn>true</alwaysOn>
-      <updateRate>30.0</updateRate>
-      <cameraName>camera/depth</cameraName>
-      <imageTopicName>depth/image_raw</imageTopicName>
-      <cameraInfoTopicName>depth/camera_info</cameraInfoTopicName>
-      <frameName>camera_link</frameName>
+      <depthImageTopicName>depth/image_raw</depthImageTopicName>
+      <depthImageCameraInfoTopicName>depth/camera_info</depthImageCameraInfoTopicName>
+      <pointCloudTopicName>depth/points</pointCloudTopicName>
+      <frameName>camera_depth_optical_frame</frameName>
+      <pointCloudCutoff>0.5</pointCloudCutoff>
+      <pointCloudCutoffMax>3.0</pointCloudCutoffMax>
+      <distortionK1>0.0</distortionK1>
+      <distortionK2>0.0</distortionK2>
+      <distortionK3>0.0</distortionK3>
+      <distortionT1>0.0</distortionT1>
+      <distortionT2>0.0</distortionT2>
+      <CxPrime>0</CxPrime>
+      <Cx>0</Cx>
+      <Cy>0</Cy>
+      <focalLength>0</focalLength>
+      <hackBaseline>0</hackBaseline>
     </plugin>
   </sensor>

Commit message: Updated readme

File: jackal_description/urdf/jackal.urdf.xacro (robot description, xacro)
@@ -234,5 +234,5 @@
   <sensor name="realsense_rgbd" type="depth">
     <always_on>true</always_on>
-    <update_rate>30</update_rate>
+    <update_rate>20</update_rate>
     <visualize>true</visualize>
     <pose>0 0 0 0 0 0</pose>
@@ -252,5 +252,5 @@
       <baseline>0.2</baseline>
       <alwaysOn>true</alwaysOn>
-      <updateRate>30.0</updateRate>
+      <updateRate>20.0</updateRate>
       <cameraName>camera</cameraName>
       <imageTopicName>color/image_raw</imageTopicName>
@@ -276,5 +276,5 @@
 </gazebo>
 <!-- IMU frame -->
-<link name="camera_imu_frame"/>
+<!-- <link name="camera_imu_frame"/>
 <joint name="camera_imu_joint" type="fixed">
   <parent link="camera_link"/>
@@ -294,5 +294,5 @@
       <headingGaussianNoise>0.005</headingGaussianNoise>
     </plugin>
-  </gazebo>
+  </gazebo> -->
 <!-- Front Lidar -->
   <joint name="lidar_front_joint" type="fixed">
